File: PCBDesign/AnalogFNN/VariableWeights.kicad_sch (KiCad schematic)
At the start: 0 parts

Commit message: Footprint updates and redid NN in/out layers
Other:
- added sheet NeuronWeightCtrl31 (NeuronWeightControl.kicad_sch)
- added sheet NeuronWeightCtrl32 (NeuronWeightControl.kicad_sch)
- sheet WeightCtrlChipSel ports: added CS1110, CS1111, CS1112, CS117, CS118, CS119, CS1210, CS1211, CS1212, CS127, CS128, CS129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; removed CS531, CS532, CS533, CS534, CS535, CS536, CS541, CS542, CS543, CS544, CS545, CS546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
