File: PCBDesign/AnalogFNN/WeightCtrlChipSel.kicad_sch (KiCad schematic)
At the start: 13 parts, among them U355 CD74HC4067SM

Commit message: Finished manual routing, working on autorouting
Connections:
- net CS111: now also U355.2 (I7); no longer U355.9 (I0)
- net CS112: now also U355.3 (I6); no longer U355.8 (I1)
- net CS113: now also U355.4 (I5); no longer U355.7 (I2)
- net CS114: now also U355.5 (I4); no longer U355.6 (I3)
- net CS115: now also U355.6 (I3); no longer U355.5 (I4)
- net CS116: now also U355.7 (I2); no longer U355.4 (I5)
- net CS121: now also U355.8 (I1); no longer U355.3 (I6)
- net CS122: now also U355.9 (I0); no longer U355.2 (I7)
- net CS135: now also U355.2 (I7); no longer U355.9 (I0)
- net CS136: now also U355.3 (I6); no longer U355.8 (I1)
- net CS141: now also U355.4 (I5); no longer U355.7 (I2)
- net CS142: now also U355.5 (I4); no longer U355.6 (I3)
- net CS143: now also U355.6 (I3); no longer U355.5 (I4)
- net CS144: now also U355.7 (I2); no longer U355.4 (I5)
- net CS145: now also U355.8 (I1); no longer U355.3 (I6)
- net CS146: now also U355.9 (I0); no longer U355.2 (I7)
- net CS163: now also U355.2 (I7); no longer U355.9 (I0)
- net CS164: now also U355.3 (I6); no longer U355.8 (I1)
- net CS165: now also U355.4 (I5); no longer U355.7 (I2)
- net CS166: now also U355.5 (I4); no longer U355.6 (I3)
- net CS211: now also U355.6 (I3); no longer U355.5 (I4)
- net CS212: now also U355.7 (I2); no longer U355.4 (I5)
- net CS213: now also U355.8 (I1); no longer U355.3 (I6)
- net CS214: now also U355.9 (I0); no longer U355.2 (I7)
- net CS231: now also U355.2 (I7); no longer U355.9 (I0)
- net CS232: now also U355.3 (I6); no longer U355.8 (I1)
- net CS233: now also U355.4 (I5); no longer U355.7 (I2)
- net CS234: now also U355.5 (I4); no longer U355.6 (I3)
- net CS235: now also U355.6 (I3); no longer U355.5 (I4)
- net CS236: now also U355.7 (I2); no longer U355.4 (I5)
- net CS241: now also U355.8 (I1); no longer U355.3 (I6)
- net CS242: now also U355.9 (I0); no longer U355.2 (I7)
- net CS255: now also U355.2 (I7); no longer U355.9 (I0)
- net CS256: now also U355.3 (I6); no longer U355.8 (I1)
- net CS261: now also U355.4 (I5); no longer U355.7 (I2)
- net CS262: now also U355.5 (I4); no longer U355.6 (I3)
- net CS263: now also U355.6 (I3); no longer U355.5 (I4)
- net CS264: now also U355.7 (I2); no longer U355.4 (I5)
- net CS265: now also U355.8 (I1); no longer U355.3 (I6)
- net CS266: now also U355.9 (I0); no longer U355.2 (I7)
- net CS323: now also U355.2 (I7); no longer U355.9 (I0)
- net CS324: now also U355.3 (I6); no longer U355.8 (I1)
- net CS325: now also U355.4 (I5); no longer U355.7 (I2)
- net CS326: now also U355.5 (I4); no longer U355.6 (I3)
- net CS331: now also U355.6 (I3); no longer U355.5 (I4)
- net CS332: now also U355.7 (I2); no longer U355.4 (I5)
- net CS333: now also U355.8 (I1); no longer U355.3 (I6)
- net CS334: now also U355.9 (I0); no longer U355.2 (I7)
- net CS351: now also U355.2 (I7); no longer U355.9 (I0)
- net CS352: now also U355.3 (I6); no longer U355.8 (I1)
- net CS353: now also U355.4 (I5); no longer U355.7 (I2)
- net CS354: now also U355.5 (I4); no longer U355.6 (I3)
- net CS355: now also U355.6 (I3); no longer U355.5 (I4)
- net CS356: now also U355.7 (I2); no longer U355.4 (I5)
- net CS361: now also U355.8 (I1); no longer U355.3 (I6)
- net CS362: now also U355.9 (I0); no longer U355.2 (I7)
- net CS415: now also U355.2 (I7); no longer U355.9 (I0)
- net CS416: now also U355.3 (I6); no longer U355.8 (I1)
- net CS421: now also U355.4 (I5); no longer U355.7 (I2)
- net CS422: now also U355.5 (I4); no longer U355.6 (I3)
- net CS423: now also U355.6 (I3); no longer U355.5 (I4)
- net CS424: now also U355.7 (I2); no longer U355.4 (I5)
- net CS425: now also U355.8 (I1); no longer U355.3 (I6)
- net CS426: now also U355.9 (I0); no longer U355.2 (I7)
- net CS443: now also U355.2 (I7); no longer U355.9 (I0)
- net CS444: now also U355.3 (I6); no longer U355.8 (I1)
- net CS445: now also U355.4 (I5); no longer U355.7 (I2)
- net CS446: now also U355.5 (I4); no longer U355.6 (I3)
- net CS451: now also U355.6 (I3); no longer U355.5 (I4)
- net CS452: now also U355.7 (I2); no longer U355.4 (I5)
- net CS453: now also U355.8 (I1); no longer U355.3 (I6)
- net CS454: now also U355.9 (I0); no longer U355.2 (I7)
- net CS511: now also U355.2 (I7); no longer U355.9 (I0)
- net CS512: now also U355.3 (I6); no longer U355.8 (I1)
- net CS513: now also U355.4 (I5); no longer U355.7 (I2)
- net CS514: now also U355.5 (I4); no longer U355.6 (I3)
- net CS515: now also U355.6 (I3); no longer U355.5 (I4)
- net CS516: now also U355.7 (I2); no longer U355.4 (I5)
- net CS521: now also U355.8 (I1); no longer U355.3 (I6)
- net CS522: now also U355.9 (I0); no longer U355.2 (I7)
- net CS535: now also U355.2 (I7); no longer U355.9 (I0)
- net CS536: now also U355.3 (I6); no longer U355.8 (I1)
- net CS541: now also U355.4 (I5); no longer U355.7 (I2)
- net CS542: now also U355.5 (I4); no longer U355.6 (I3)
- net CS543: now also U355.6 (I3); no longer U355.5 (I4)
- net CS544: now also U355.7 (I2); no longer U355.4 (I5)
- net CS545: now also U355.8 (I1); no longer U355.3 (I6)
- net CS546: now also U355.9 (I0); no longer U355.2 (I7)

Commit message: Footprint updates and redid NN in/out layers
Connections:
- net CS1612: now reaches U355.16 (I15)
- net CS1611: now reaches U355.17 (I14)
- net CS1610: now reaches U355.18 (I13)
- net CS169: now reaches U355.19 (I12)
- net CS1510: now reaches U355.2 (I7)
- net CS168: now reaches U355.20 (I11)
- net CS167: now reaches U355.21 (I10)
- net CS1512: now reaches U355.22 (I9)
- net CS1511: now reaches U355.23 (I8)
- net CS159: now reaches U355.3 (I6)
- net CS158: now reaches U355.4 (I5)
- net CS157: now reaches U355.5 (I4)
- net CS531 renamed CS117
- net CS532 renamed CS118
- net CS533 renamed CS119
- net CS534 renamed CS1110
- net CS535 renamed CS1212
- net CS536 renamed CS1211
- net CS541 renamed CS1210
- net CS542 renamed CS129
- net CS543 renamed CS128
- net CS544 renamed CS127
- net CS545 renamed CS1112
- net CS546 renamed CS1111
- net CS551 renamed CS137
- net CS552 renamed CS138
- net CS553 renamed CS139
- net CS554 renamed CS1310
- net CS555 renamed CS1311
- net CS556 renamed CS1312
- net CS561 renamed CS147
- net CS562 renamed CS148
- net CS563 renamed CS149
- net CS564 renamed CS1410
- net CS565 renamed CS1411
- net CS566 renamed CS1412
