File: PCBDesign/AnalogFNN/Adder.kicad_sch (KiCad schematic)
At the start: 9 parts, among them U27 TLV9004xRUCR

Commit message: Footprint updates and redid NN in/out layers
Parts:
- C20: footprint Capacitor_SMD:C_0201_0603Metric -> Capacitor_SMD:C_0603_1608Metric
